File: HW2/JiaruiYang_ME433_HW2/JY_HW2_Sche.sch (EAGLE design)
At the start: 22 parts, among them J1 USB-MB-H

Commit message: finish sche
Connections:
- new net N$2: LED2.C, R2.2
- net +3V3: now also J3.2, R3.2, R4.2
- net +5V: now also J2.2
- net A0: now also J3.8
- net A1: now also J3.7
- net A4/LED: now also J3.3, LED2.A
- net B13: now also J2.6
- net B14: now also J2.7
- net B15: now also J2.8
- net B2: now also J3.6
- net B3: now also J3.5
- net B4/USER: now also J3.4, R4.1, U$5.2
- net B7: now also J2.3
- net B8: now also J2.4
- net B9: now also J2.5
- net D+: now also J1.D+
- net D-: now also J1.D-
- net GND: now also J2.1, J3.1, R2.1, U$4.1, U$5.1
- net MCLR: now also R3.1, U$4.2
- net USBID: now also J1.ID
Other:
- moved on the sheet: R4, U$4, U$5
Changed lines of the file:
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@@
 <instance part="LED1" gate="G$1" x="167.64" y="104.14"/>
 <instance part="LED2" gate="G$1" x="185.42" y="104.14"/>
-<instance part="U$4" gate="G$1" x="182.88" y="63.5"/>
-<instance part="U$5" gate="G$1" x="182.88" y="43.18"/>
+<instance part="U$4" gate="G$1" x="190.5" y="66.04"/>
+<instance part="U$5" gate="G$1" x="190.5" y="40.64"/>
 <instance part="R1" gate="G$1" x="167.64" y="91.44" rot="R90"/>
 <instance part="R2" gate="G$1" x="185.42" y="91.44" rot="R90"/>
 <instance part="R3" gate="G$1" x="203.2" y="78.74" rot="R90"/>
-<instance part="R4" gate="G$1" x="203.2" y="53.34" rot="R90"/>
+<instance part="R4" gate="G$1" x="203.2" y="50.8" rot="R90"/>
 <instance part="C1" gate="G$1" x="93.98" y="63.5"/>
 <instance part="C2" gate="G$1" x="12.7" y="2.54"/>
@@
 <instance part="GND12" gate="1" x="139.7" y="91.44"/>
 <instance part="GND13" gate="1" x="147.32" y="91.44"/>
-<instance part="GND14" gate="1" x="203.2" y="63.5"/>
-<instance part="GND15" gate="1" x="203.2" y="40.64"/>
+<instance part="GND14" gate="1" x="170.18" y="63.5"/>
+<instance part="GND15" gate="1" x="170.18" y="38.1"/>
 <instance part="GND16" gate="1" x="167.64" y="81.28"/>
 <instance part="GND17" gate="1" x="185.42" y="81.28"/>
-<instance part="GND18" gate="1" x="165.1" y="17.78"/>
-<instance part="GND19" gate="1" x="165.1" y="-12.7"/>
+<instance part="GND18" gate="1" x="157.48" y="12.7"/>
+<instance part="GND19" gate="1" x="157.48" y="-17.78"/>
 <instance part="P+1" gate="1" x="88.9" y="109.22" rot="MR0"/>
 <instance part="P+2" gate="1" x="83.82" y="2.54" rot="MR0"/>
@@
 <instance part="+3V3" gate="G$1" x="203.2" y="91.44"/>
 <instance part="+3V4" gate="G$1" x="154.94" y="111.76"/>
-<instance part="+3V5" gate="G$1" x="213.36" y="58.42"/>
-<instance part="+3V6" gate="G$1" x="165.1" y="-5.08"/>
-<instance part="P+3" gate="1" x="165.1" y="25.4" rot="MR0"/>
+<instance part="+3V5" gate="G$1" x="203.2" y="63.5"/>
+<instance part="+3V6" gate="G$1" x="170.18" y="-10.16" rot="MR0"/>
+<instance part="P+3" gate="1" x="170.18" y="20.32" rot="MR0"/>
 <instance part="+3V7" gate="G$1" x="101.6" y="43.18" rot="MR0"/>
 <instance part="+3V8" gate="G$1" x="109.22" y="63.5"/>
@@
 <pinref part="GND6" gate="1" pin="GND"/>
 <wire x1="121.92" y1="55.88" x2="109.22" y2="55.88" width="0.1524" layer="91"/>
+</segment>
+<segment>
+<pinref part="R2" gate="G$1" pin="1"/>
+<pinref part="GND17" gate="1" pin="GND"/>
+<wire x1="185.42" y1="86.36" x2="185.42" y2="83.82" width="0.1524" layer="91"/>
+</segment>
+<segment>
+<pinref part="U$5" gate="G$1" pin="1"/>
+<pinref part="GND15" gate="1" pin="GND"/>
+<wire x1="177.8" y1="40.64" x2="170.18" y2="40.64" width="0.1524" layer="91"/>
+</segment>
+<segment>
+<pinref part="GND14" gate="1" pin="GND"/>
+<pinref part="U$4" gate="G$1" pin="1"/>
+<wire x1="170.18" y1="66.04" x2="177.8" y2="66.04" width="0.1524" layer="91"/>
+</segment>
+<segment>
+<pinref part="J2" gate="G$1" pin="1"/>
+<pinref part="GND18" gate="1" pin="GND"/>
+<wire x1="154.94" y1="15.24" x2="157.48" y2="15.24" width="0.1524" layer="91"/>
+</segment>
+<segment>
+<pinref part="J3" gate="G$1" pin="1"/>
+<pinref part="GND19" gate="1" pin="GND"/>
+<wire x1="154.94" y1="-15.24" x2="157.48" y2="-15.24" width="0.1524" layer="91"/>
 </segment>
 </net>
@@
 <pinref part="U$1" gate="G$1" pin="15.VBUS"/>
 <wire x1="83.82" y1="0" x2="76.2" y2="0" width="0.1524" layer="91"/>
+</segment>
+<segment>
+<pinref part="J2" gate="G$1" pin="2"/>
+<pinref part="P+3" gate="1" pin="+5V"/>
+<wire x1="154.94" y1="17.78" x2="170.18" y2="17.78" width="0.1524" layer="91"/>
 </segment>
 </net>
@@
 <wire x1="109.22" y1="60.96" x2="121.92" y2="60.96" width="0.1524" layer="91"/>
 </segment>
+<segment>
+<pinref part="+3V5" gate="G$1" pin="+3V3"/>
+<pinref part="R4" gate="G$1" pin="2"/>
+<wire x1="203.2" y1="60.96" x2="203.2" y2="55.88" width="0.1524" layer="91"/>
+</segment>
+<segment>
+<pinref part="R3" gate="G$1" pin="2"/>
+<pinref part="+3V3" gate="G$1" pin="+3V3"/>
+<wire x1="203.2" y1="83.82" x2="203.2" y2="88.9" width="0.1524" layer="91"/>
+</segment>
+<segment>
+<pinref part="J3" gate="G$1" pin="2"/>
+<pinref part="+3V6" gate="G$1" pin="+3V3"/>
+<wire x1="154.94" y1="-12.7" x2="170.18" y2="-12.7" width="0.1524" layer="91"/>
+</segment>
 </net>
 <net name="N$3" class="0">
@@
 <label x="114.3" y="66.04" size="1.778" layer="95"/>
 </segment>
+<segment>
+<pinref part="U$4" gate="G$1" pin="2"/>
+<pinref part="R3" gate="G$1" pin="1"/>
+<wire x1="203.2" y1="66.04" x2="203.2" y2="73.66" width="0.1524" layer="91"/>
+<wire x1="203.2" y1="66.04" x2="215.9" y2="66.04" width="0.1524" layer="91"/>
+<junction x="203.2" y="66.04"/>
+<label x="210.82" y="66.04" size="1.778" layer="95"/>
+</segment>
 </net>
 <net name="A0" class="0">
@@
 <label x="15.24" y="60.96" size="1.778" layer="95"/>
 </segment>
+<segment>
+<pinref part="J3" gate="G$1" pin="8"/>
+<wire x1="154.94" y1="2.54" x2="165.1" y2="2.54" width="0.1524" layer="91"/>
+<label x="160.02" y="2.54" size="1.778" layer="95"/>
+</segment>
 </net>
 <net name="A1" class="0">
@@
 <label x="15.24" y="55.88" size="1.778" layer="95"/>
 </segment>
+<segment>
+<pinref part="J3" gate="G$1" pin="7"/>
+<wire x1="154.94" y1="0" x2="165.1" y2="0" width="0.1524" layer="91"/>
+<label x="160.02" y="0" size="1.778" layer="95"/>
+</segment>
 </net>
 <net name="PGD" class="0">
@@
 <label x="15.24" y="40.64" size="1.778" layer="95"/>
 </segment>
+<segment>
+<pinref part="J3" gate="G$1" pin="6"/>
+<wire x1="154.94" y1="-2.54" x2="165.1" y2="-2.54" width="0.1524" layer="91"/>
+<label x="160.02" y="-2.54" size="1.778" layer="95"/>
+</segment>
 </net>
 <net name="B3" class="0">
@@
 <label x="15.24" y="35.56" size="1.778" layer="95"/>
 </segment>
+<segment>
+<pinref part="J3" gate="G$1" pin="5"/>
+<wire x1="154.94" y1="-5.08" x2="165.1" y2="-5.08" width="0.1524" layer="91"/>
+<label x="160.02" y="-5.08" size="1.778" layer="95"/>
+</segment>
 </net>
 <net name="B4/USER" class="0">
@@
 <label x="15.24" y="15.24" size="1.778" layer="95"/>
 </segment>
+<segment>
+<pinref part="R4" gate="G$1" pin="1"/>
+<pinref part="U$5" gate="G$1" pin="2"/>
+<wire x1="203.2" y1="45.72" x2="203.2" y2="40.64" width="0.1524" layer="91"/>
+<wire x1="203.2" y1="40.64" x2="215.9" y2="40.64" width="0.1524" layer="91"/>
+<junction x="203.2" y="40.64"/>
+<label x="210.82" y="40.64" size="1.778" layer="95"/>
+</segment>
+<segment>
+<pinref part="J3" gate="G$1" pin="4"/>
+<wire x1="154.94" y1="-7.62" x2="165.1" y2="-7.62" width="0.1524" layer="91"/>
+<label x="160.02" y="-7.62" size="1.778" layer="95"/>
+</segment>
 </net>
 <net name="A4/LED" class="0">
@@
 <label x="15.24" y="10.16" size="1.778" layer="95"/>
 </segment>
+<segment>
+<pinref part="LED2" gate="G$1" pin="A"/>
+<wire x1="185.42" y1="106.68" x2="185.42" y2="119.38" width="0.1524" layer="91"/>
+<label x="185.42" y="111.76" size="1.778" layer="95" rot="R90"/>
+</segment>
+<segment>
+<pinref part="J3" gate="G$1" pin="3"/>
+<wire x1="154.94" y1="-10.16" x2="165.1" y2="-10.16" width="0.1524" layer="91"/>
+<label x="160.02" y="-10.16" size="1.778" layer="95"/>
+</segment>
 </net>
 <net name="USBID" class="0">
@@
 <label x="20.32" y="0" size="1.778" layer="95"/>
 </segment>
+<segment>
+<pinref part="J1" gate="G$1" pin="ID"/>
+<wire x1="35.56" y1="101.6" x2="43.18" y2="101.6" width="0.1524" layer="91"/>
+<label x="38.1" y="101.6" size="1.778" layer="95"/>
+</segment>
 </net>
 <net name="B15" class="0">
@@
 <label x="81.28" y="55.88" size="1.778" layer="95"/>
 </segment>
+<segment>
+<pinref part="J2" gate="G$1" pin="8"/>
+<wire x1="154.94" y1="33.02" x2="165.1" y2="33.02" width="0.1524" layer="91"/>
+<label x="160.02" y="33.02" size="1.778" layer="95"/>
+</segment>
 </net>
 <net name="B14" class="0">
@@
 <label x="81.28" y="50.8" size="1.778" layer="95"/>
 </segment>
+<segment>
+<pinref part="J2" gate="G$1" pin="7"/>
+<wire x1="154.94" y1="30.48" x2="165.1" y2="30.48" width="0.1524" layer="91"/>
+<label x="160.02" y="30.48" size="1.778" layer="95"/>
+</segment>
 </net>
 <net name="B13" class="0">
@@
 <label x="81.28" y="45.72" size="1.778" layer="95"/>
 </segment>
+<segment>
+<pinref part="J2" gate="G$1" pin="6"/>
+<wire x1="154.94" y1="27.94" x2="165.1" y2="27.94" width="0.1524" layer="91"/>
+<label x="160.02" y="27.94" size="1.778" layer="95"/>
+</segment>
 </net>
 <net name="D-" class="0">
@@
 <label x="81.28" y="35.56" size="1.778" layer="95"/>
 </segment>
+<segment>
+<pinref part="J1" gate="G$1" pin="D-"/>
+<wire x1="35.56" y1="96.52" x2="43.18" y2="96.52" width="0.1524" layer="91"/>
+<label x="38.1" y="96.52" size="1.778" layer="95"/>
+</segment>
 </net>
 <net name="D+" class="0">
@@
 <label x="81.28" y="30.48" size="1.778" layer="95"/>
 </segment>
+<segment>
+<pinref part="J1" gate="G$1" pin="D+"/>
+<wire x1="35.56" y1="99.06" x2="43.18" y2="99.06" width="0.1524" layer="91"/>
+<label x="38.1" y="99.06" size="1.778" layer="95"/>
+</segment>
 </net>
 <net name="B9" class="0">
@@
 <label x="81.28" y="15.24" size="1.778" layer="95"/>
 </segment>
+<segment>
+<pinref part="J2" gate="G$1" pin="5"/>
+<wire x1="154.94" y1="25.4" x2="165.1" y2="25.4" width="0.1524" layer="91"/>
+<label x="160.02" y="25.4" size="1.778" layer="95"/>
+</segment>
 </net>
 <net name="B8" class="0">
@@
 <label x="81.28" y="10.16" size="1.778" layer="95"/>
 </segment>
+<segment>
+<pinref part="J2" gate="G$1" pin="4"/>
+<wire x1="154.94" y1="22.86" x2="165.1" y2="22.86" width="0.1524" layer="91"/>
+<label x="160.02" y="22.86" size="1.778" layer="95"/>
+</segment>
 </net>
 <net name="B7" class="0">
@@
 <label x="81.28" y="5.08" size="1.778" layer="95"/>
 </segment>
-</net>
+<segment>
+<pinref part="J2" gate="G$1" pin="3"/>
+<wire x1="154.94" y1="20.32" x2="165.1" y2="20.32" width="0.1524" layer="91"/>
+<label x="160.02" y="20.32" size="1.778" layer="95"/>
+</segment>
+</net>
+<net name="N$2" class="0">
+<segment>
+<pinref part="LED2" gate="G$1" pin="C"/>
+<pinref part="R2" gate="G$1" pin="2"/>
+<wire x1="185.42" y1="99.06" x2="185.42" y2="96.52" width="0.1524" layer="91"/>
+</segment>
+</net>
